File: Hardware/Basic/Bottom/Omni-BASIC-BOTTOM.brd (EAGLE design)
At the start: 33 x 33 mm, 32 parts, among them U1 AD5242-SO16

Commit message: Latest Update
Parts:
- moved C24 35.9 mm to (27.4, 32.3)
- moved IMU1 35.7 mm to (31.6, 32.5)
- moved R23 27.5 mm to (29.8, 19.7), turned to 180 degrees
- moved C19 25.9 mm to (29.8, 18.4), turned to 180 degrees
- moved C10 25.6 mm to (5.22, 28.9)
- moved R21 25.0 mm to (32.6, 15.1), turned to 270 degrees
- moved R22 24.3 mm to (29.8, 17.0), turned to 0 degrees
- moved C16 23.8 mm to (33.9, 12.1), turned to 90 degrees
- moved R15 22.3 mm to (32.6, 12.1), turned to 270 degrees
- moved R18 22.3 mm to (25.4, 17.9), turned to 270 degrees
- moved R17 21.8 mm to (24.3, 17.9), turned to 90 degrees
- moved R19 21.3 mm to (33.4, 8.98), turned to 270 degrees
- moved C18 21.1 mm to (8.37, 6.62)
- moved U1 21.0 mm to (13.4, 8.38)
- moved R20 17.8 mm to (30.5, 5.41), turned to 180 degrees
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Routing:
- net A7/PPG: track 2.11 -> 12.6 mm
- net G.W2: track 3.22 -> 12.6 mm, vias 0 -> 2
- net N$13: track 0.00 -> 4.93 mm
- net N$15: track 0.00 -> 4.70 mm
- net N$16: track 0.00 -> 3.49 mm
- net GND: track 3.69 -> 7.07 mm, vias 3 -> 6

Commit message: Latest Update
Parts:
- removed OP4: (no value), LinnesLab-AnalogIC:SOT23-5
- removed U$4: AD5171, LinnesLab-DigitalIC:SOT-23-8
- added AD5171: AD5171, LinnesLab-DigitalIC:SOT-23-8
- added C1: 100n, LinnesLab-Passives:C0603
- added C2, C3, C6: 1u, LinnesLab-Passives:C0603
- added C4, C7: 4.7u, LinnesLab-Passives:C0603
- added CHRG1: MCP73831, LinnesLab-Power:SOT23-5
- added LDO1: MIC5504, LinnesLab-Power:SOT23-5
- added R3, R6, R7: 100k, LinnesLab-Passives:R0603
- added R4: (no value), LinnesLab-Passives:R0603
- added TIA: (no value), LinnesLab-AnalogIC:SOT23-5
- added U2: PCF8523, LinnesLab-Clocks:SO8
- added XTAL2: 32.7680kHz, LinnesLab-Clocks:2-SMD.NOLEAD.2.0MMTO1.2MM
- J1: device LinnesLab-Connectors:1X07 -> LinnesLab-Connectors:1X07_1.27MM
- moved IMU1 25.5 mm to (6.21, 29.4), turned to 90 degrees
- moved C22 22.3 mm to (14.5, 21.5)
- moved C24 21.7 mm to (6.69, 25.9), turned to 0 degrees
- moved C10 15.2 mm to (16.7, 18.8), turned to 180 degrees
- moved R16 13.3 mm to (19.0, 28.5)
- moved C17 8.02 mm to (6.69, 24.6), turned to 0 degrees
- moved C16 5.19 mm to (33.4, 17.2)
- moved R15 5.18 mm to (32.1, 17.2)
- moved R21 5.12 mm to (32.8, 20.2)
- moved Q1 4.52 mm to (19.0, 26.3), turned to 180 degrees
- moved R19 4.36 mm to (33.8, 13.3)
- moved C18 1.04 mm to (8.63, 7.63), turned to 270 degrees
- renumbered U1 to AD5242
Connections:
- removed net N$7: J1.1
- new net A4/BATTERY_STATUS: R6.1, R7.2
- new net D27/CHARGE_STATUS: CHRG1.1, R3.1
- new net N$3: U2.2, XTAL2.P$1
- new net VBATT: U2.3
- new net VIN1: C4.2, CHRG1.4, R3.2
- new net VLIPO: C7.1, CHRG1.3, R6.2
- net 3.3V: now also AD5171.2, AD5171.6, C2.1, C6.1, J1.4, LDO1.5, TIA.5, U2.8; no longer OP4.5, U$4.2, U$4.6
- net A6/TIA: now also J1.6, TIA.1; no longer J1.5, OP4.1
- net D29/LED.CONTROL: now also AD5171.8, J1.5; no longer J1.6, U$4.8
- net GND: now also AD5171.3, C1.1, C2.2, C3.1, C4.1, C6.2, C7.2, CHRG1.2, J1.3, LDO1.2, R4.1, R7.1, TIA.2, TIA.3, U2.4; no longer OP4.2, OP4.3, U$4.3
- net N$4: now also U2.1, XTAL2.P$2; no longer J1.4
- net N$5: now also CHRG1.5, R4.2; no longer J1.3
- net N$6: now also C3.2, LDO1.1, LDO1.3; no longer J1.2
- net N$9: now also AD5171.1, AD5171.7; no longer U$4.1, U$4.7
- net PD.C: now also TIA.4; no longer OP4.4
- net SCL: now also AD5171.4, J1.2, U2.6; no longer U$4.4
- net SDA: now also AD5171.5, J1.1, U2.5; no longer U$4.5
- net VREF: now also C1.2
Routing:
- net A6/TIA: track 0.00 -> 62.1 mm, vias 0 -> 2
- net SDA: track 0.00 -> 35.9 mm
- net SCL: track 0.00 -> 33.9 mm, vias 0 -> 2
- net A7/PPG: track 12.6 -> 43.9 mm
- net VREF: track 1.27 -> 32.5 mm, vias 0 -> 8
- net 3.3V: track 0.00 -> 31.0 mm, vias 0 -> 4
- net PD.C: track 0.00 -> 18.9 mm
- net GND: track 7.07 -> 23.9 mm, vias 6 -> 13
- net N$9: track 0.00 -> 15.9 mm
- net D29/LED.CONTROL: track 0.00 -> 14.4 mm, vias 0 -> 2
- net N$13: track 4.93 -> 18.5 mm, vias 0 -> 2
- net N$16: track 3.49 -> 11.0 mm
- net N$17: track 21.3 -> 18.0 mm
- net N$8: track 0.00 -> 1.24 mm
- net LED.C: track 0.00 -> 1.15 mm
