File: Hardware/Basic/Top/Omni-BASIC-TOP.sch (EAGLE design)
At the start: 29 parts, among them U2 NRF52832_MODULE_MDBT42

Commit message: commit operation
Parts:
- added C2, C5, C6: 1u, LinnesLab-Passives:CAPACITOR0603
- added C20, C21: 4.7u, LinnesLab-Passives:CAPACITOR0603
- added C22: 100n, LinnesLab-Passives:CAPACITOR0603
- added C23, C24: 47p, LinnesLab-Passives:CAPACITOR0603
- added CHRG2: MCP73831, LinnesLab-Power:MCP73831
- added D4, D5: (no value), LinnesLab-DiscreteSemi:SCHOTTKY-USC
- added J1: (no value), LinnesLab-Connectors:CONN_07
- added J2: (no value), LinnesLab-Connectors:CONN_02
- added JP2: (no value), LinnesLab-Switches:JUMPER-SMT_2_NO_SILK
- added LDO2: MIC5504, LinnesLab-Power:MIC5504
- added LED5: RED, LinnesLab-LED:LED0603
- added LED6: YELLOW, LinnesLab-LED:LED0603
- added R1, R2: 10k, LinnesLab-Passives:RESISTOR0603
- added R11: (no value), LinnesLab-Passives:RESISTOR0603
- added R12, R13, R14, R15: 100k, LinnesLab-Passives:RESISTOR0603
- added R17, R18: 27, LinnesLab-Passives:RESISTOR0603
- added R19, R20: 1k, LinnesLab-Passives:RESISTOR0603
- added R21, R22: 0, LinnesLab-Passives:RESISTOR0603
- added SW1, SW2: SWITCH.MOM, LinnesLab-Switches:SWITCH.MOM
- added U4: PCF8523, LinnesLab-Clocks:PCF8523
- added U5: FT231XS, LinnesLab-DigitalIC:FT231XS
- added USB2: USB.MICRO-BIGGERPADS, LinnesLab-Connectors:USB.MICRO-BIGGERPADS
- added XTAL3: 32.7680kHz, LinnesLab-Clocks:CRYSTALECS-.327-12.5-12-C-TR
- C13, C15, C16, C17, C18, C19: SPICEPREFIX (none) -> C
- R6, R7: SPICEPREFIX (none) -> R
- U3: SPICEPREFIX (none) -> X
Connections:
- removed net CD1: SD2.CARD_DETECT
- removed net CS.OLED: U3./CS
- removed net DC.OLED: U3.DC/I2C_SA0
- removed net RESET.OLED: U3./RES
- removed net RXD: U2.P0.08
- removed net SD.CS: SD2.CS
- removed net TXD: U2.P0.06
- new net !CTS: JP2.2, U5.!CTS
- new net !DTR: U5.!DTR
- new net A4/BATTERY_STATUS: R13.1, R14.2, U2.P0.28/AIN4
- new net A6/TIA: J1.5, U2.P0.30/AIN6
- new net A7/PPG: J1.7, U2.P0.31/AIN7
- new net D11/SW1: SW1.1, U2.P0.11
- new net D15/SW2: SW2.1, U2.P0.15
- new net D16/CS.OLED: U2.P0.16, U3./CS
- new net D27/CHARGE_STATUS: CHRG2.STAT, R12.1, U2.P0.27
- new net D29/LED.CONTROL: J1.6, U2.P0.29/AIN5
- new net D3/RESET.OLED: U2.P0.03/AIN1, U3./RES
- new net D4/DC.OLED: U2.P0.04/AIN2, U3.DC/I2C_SA0
- new net D5/CD1: SD2.CARD_DETECT, U2.P0.05/AIN3
- new net D7/SD.CS: SD2.CS, U2.P0.07
- new net FT3V3: U5.3V3OUT
- new net N$17: CHRG2.PROG, R11.2
- new net N$19: U4.OSCO, XTAL3.1
- new net N$20: U4.OSCI, XTAL3.2
- new net N$23: R17.2, U5.USBDM
- new net N$24: R18.2, U5.USBDP
- new net N$25: LED5.C, R19.2
- new net N$26: LED6.C, R20.2
- new net RXD.FT: R22.1, U5.RXD
- new net RXD.NRF: R21.2, U2.P0.08
- new net RXLED: R19.1, U5.CBUS1
- new net TXD.FT: R21.1, U5.TXD
- new net TXD.NRF: R22.2, U2.P0.06
- new net TXLED: R20.1, U5.CBUS2
- new net USB+: C23.1, R18.1, USB2.D+
- new net USB-: C24.2, R17.1, USB2.D-
- new net VBATT: U4.VBAT
- new net VIN: C21.2, C5.2, CHRG2.VIN, D4.C, D5.C, LDO2.EN, LDO2.IN, R12.2
- new net VLIPO: C20.1, CHRG2.VBAT, D4.A, J2.2, R13.2
- new net V_USB: D5.A, U5.VCC, USB2.V+
- net 3.3V: now also C2.1, C22.2, C6.1, LDO2.OUT, LED5.A, LED6.A, R1.2, R15.2, R2.2, U4.VDD, U5.!RESET, U5.VCCIO
- net GND: now also C2.2, C20.2, C21.1, C22.1, C23.2, C24.1, C5.1, C6.2, CHRG2.VSS, J2.1, JP2.1, LDO2.GND, R11.1, R14.1, R15.1, SW1.3, SW1.4, SW2.3, SW2.4, U4.VSS, U5.GND@16, U5.GND@6, USB2.GND
- net SCL: now also R2.1, U4.SCL
- net SDA: now also R1.1, U4.SDA
Other:
- note added: "Back-up battery if desired"
- note added: "I don't remember if CTS needs to be grounded or left floating so here's a jumper to ground so it can be configued either way dynamically."
- note added: "I2C Address = 0x68h"
- note added: "TXD goes to RX on the other device RXD goes to TX on the other device"
- moved on the sheet: C10, C11, C12, C13, C14, C15, C16, C17, C18, C19, C7, C8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

Commit message: Latest Update
Parts:
- removed C15: 2.2uF, LinnesLab-Passives:CAPACITOR0402
- removed C2, C6: 1u, LinnesLab-Passives:CAPACITOR0603
- removed C22: 100n, LinnesLab-Passives:CAPACITOR0603
- removed C23, C24: 47p, LinnesLab-Passives:CAPACITOR0603
- removed CHRG2: MCP73831, LinnesLab-Power:MCP73831
- removed D4: (no value), LinnesLab-DiscreteSemi:SCHOTTKY-USC
- removed LDO2: MIC5504, LinnesLab-Power:MIC5504
- removed LED5: RED, LinnesLab-LED:LED0603
- removed LED6: YELLOW, LinnesLab-LED:LED0603
- removed R19: 1k, LinnesLab-Passives:RESISTOR0603
- removed R21, R22: 0, LinnesLab-Passives:RESISTOR0603
- removed SD2: (no value), LinnesLab-Connectors:MICROSD
- removed U5: FT231XS, LinnesLab-DigitalIC:FT231XS
- removed XTAL3: 32.7680kHz, LinnesLab-Clocks:CRYSTALECS-.327-12.5-12-C-TR
- added C4: 10u, LinnesLab-Passives:CAPACITOR0805
- added D3: (no value), LinnesLab-DiscreteSemi:SCHOTTKY-USC
- added LED1: RED, LinnesLab-LED:LED0603
- added LED2: BLUE, LinnesLab-LED:LED0603
- added SD1: (no value), LinnesLab-Connectors:MICROSD
- C11: value 300p -> 47p
- C12: value 10u -> 100n; device LinnesLab-Passives:CAPACITOR0805 -> LinnesLab-Passives:CAPACITOR0603
- C13: value 2.2uF -> 47p; device LinnesLab-Passives:CAPACITOR0402 -> LinnesLab-Passives:CAPACITOR0603; SPICEPREFIX C -> (none)
- C20, C21: value 4.7u -> 2.2uF; device LinnesLab-Passives:CAPACITOR0603 -> LinnesLab-Passives:CAPACITOR0402; SPICEPREFIX (none) -> C
- C5: value 1u -> (none)
- C9: value (none) -> 300p
- J1: device LinnesLab-Connectors:CONN_07 -> LinnesLab-Connectors:CONN_02
- J2: device LinnesLab-Connectors:CONN_02 -> LinnesLab-Connectors:CONN_07-1.27MM
- LED4: value BLUE -> YELLOW
- R11: value (none) -> 27
- R12: value 100k -> 27
- R13: value 100k -> 10k; SPICEPREFIX (none) -> R
- R14: value 100k -> 1k
- R15: value 100k -> 390k; SPICEPREFIX (none) -> R
- R17, R18: value 27 -> 0
- R6: value 10k -> 100k; SPICEPREFIX R -> (none)
- R7: value 390k -> 100k; SPICEPREFIX R -> (none)
- SW1, SW2: value SWITCH.MOM -> (none); device LinnesLab-Switches:SWITCH.MOM -> LinnesLab-Switches:SPST-PTS830GG140-COPY.1-3
- SW3, SW4: value (none) -> SWITCH.MOM; device LinnesLab-Switches:SPST-PTS830GG140-COPY.1-3 -> LinnesLab-Switches:SWITCH.MOM
- U3: value (none) -> FT231XS; device LinnesLab-Displays:DISP_OLED_UG-2864HSWEG01-NO-WRAPAROUND -> LinnesLab-DigitalIC:FT231XS; SPICEPREFIX X -> (none)
- U4: value PCF8523 -> (none); device LinnesLab-Clocks:PCF8523 -> LinnesLab-Displays:DISP_OLED_UG-2864HSWEG01-NO-WRAPAROUND; DIGIKEY 568-5306-1-ND -> (none); I2C_ADDRESS 0x68h -> (none); MFN PCF8523T/1,118 -> (none); MFN_MANUFACTURER NXP USA Inc. -> (none); SPICEPREFIX (none) -> X
- renumbered C7 to C3, CORTEX1 to DEBUG1, D5 to D2, JP2 to JP1, L2 to L1, R20 to R16, R3 to R8, R4 to R9, R5 to R10, U2 to U1, USB2 to USB1, XTAL2 to XTAL1
Connections:
- removed net N$17: CHRG2.PROG, R11.2
- removed net N$19: U4.OSCO, XTAL3.1
- removed net N$20: U4.OSCI, XTAL3.2
- removed net VBATT: U4.VBAT
- net !CTS: now also U3.!CTS; no longer U5.!CTS
- net !DTR: now also U3.!DTR; no longer U5.!DTR
- net 3.3V: now also C14.2, C20.2, C21.2, C4.2, D3.C, J2.4, LED3.A, LED4.A, SD1.VDD, U3.!RESET, U3.VCCIO, U4.VBAT; no longer C12.2, C17.2, C19.2, C2.1, C22.2, C6.1, D1.C, LDO2.OUT, LED5.A, LED6.A, R15.2, SD2.VDD, U3.VBAT, U3.VDD, U5.!RESET, U5.VCCIO
- net A4/BATTERY_STATUS: now also R6.1, R7.2; no longer R13.1, R14.2
- net A6/TIA: now also J2.6; no longer J1.5
- net A7/PPG: now also J2.7; no longer J1.7
- net CD2: now also SD1.CARD_DETECT1; no longer SD2.CARD_DETECT1
- net D11/SW1: now also SW3.1; no longer SW1.1
- net D15/SW2: now also SW4.1; no longer SW2.1
- net D16/CS.OLED: now also U4./CS; no longer U3./CS
- net D27/CHARGE_STATUS: no longer CHRG2.STAT, R12.1
- net D29/LED.CONTROL: now also J2.5; no longer J1.6
- net D3/RESET.OLED: now also U4./RES; no longer U3./RES
- net D4/DC.OLED: now also U4.DC/I2C_SA0; no longer U3.DC/I2C_SA0
- net D5/CD1: now also SD1.CARD_DETECT; no longer SD2.CARD_DETECT
- net D7/SD.CS: now also SD1.CS; no longer SD2.CS
- net DFU: now also SW1.B; no longer SW3.B
- net DTR: now also C12.1; no longer C14.1
- net FT3V3: now also U3.3V3OUT; no longer U5.3V3OUT
- net GND: now also C11.1, C13.2, C14.1, C20.1, C4.1, C8.2, J1.1, J2.3, LED1.C, LED2.C, R13.1, R15.2, R7.1, SD1.GND, SD1.GND1, SD1.VSS, SW1.A, SW2.B, SW3.3, SW4.3, U3.GND@16, U3.GND@6, U4.BS0, U4.BS2, U4.NC(GND)@1, U4.NC(GND)@2, U4.VLSS; no longer C11.2, C12.1, C17.1, C19.1, C2.2, C20.2, C22.1, C23.2, C24.1, C6.2, C8.1, CHRG2.VSS, J2.1, LDO2.GND, LED3.C, LED4.C, R11.1, R14.1, R15.1, R6.1, R7.2, SD2.GND, SD2.GND1, SD2.VSS, SW1.3, SW1.4, SW2.3, SW2.4, SW3.A, SW4.B, U3.BS0, U3.BS2, U3.NC(GND)@1, U3.NC(GND)@2, U3.VLSS, U3.VSS, U5.GND@16, U5.GND@6
- net MISO: now also SD1.DATA_OUT; no longer SD2.DATA_OUT
- net MOSI: now also SD1.DATA_IN, U4.D1/SPI_SDIN/I2C_SDA; no longer SD2.DATA_IN, U3.D1/SPI_SDIN/I2C_SDA
- net N$1: now also R13.2, U4.BS1; no longer R6.2, U3.BS1
- net N$10: now also LED2.A; no longer LED4.A
- net N$13: now also U4.VCC; no longer U3.VCC
- net N$15: now also U4.VCOMH; no longer U3.VCOMH
- net N$2: now also R15.1, U4.IREF; no longer R7.1, U3.IREF
- net N$23: now also R11.2, U3.USBDM; no longer R17.2, U5.USBDM
- net N$24: now also R12.2, U3.USBDP; no longer R18.2, U5.USBDP
- net N$25: now also LED3.C, R14.2; no longer LED5.C, R19.2
- net N$26: now also LED4.C; no longer LED6.C
- net N$3: now also C19.2, U4.C2P; no longer C13.2, U3.C2P
- net N$4: now also C5.2; no longer C8.2
- net N$5: now also C19.1, U4.C2N; no longer C13.1, U3.C2N
- net N$6: now also C8.1; no longer C9.1
- net N$7: now also C17.2, U4.C1P; no longer C15.2, U3.C1P
- net N$8: now also C17.1, U4.C1N; no longer C15.1, U3.C1N
- net N$9: now also LED1.A; no longer LED3.A
- net P0.09/NFC1: now also C9.1; no longer C11.1
- net RESET: now also C12.2, D3.A, SW2.A; no longer C14.2, D1.A, SW4.A
- net RXD.FT: now also R18.1, U3.RXD; no longer R22.1, U5.RXD
- net RXD.NRF: now also R17.2; no longer R21.2
- net RXLED: now also R14.1, U3.CBUS1; no longer R19.1, U5.CBUS1
- net SCK: now also SD1.SCLK, U4.D0/SPI_SCLK/I2C_SCK; no longer SD2.SCLK, U3.D0/SPI_SCLK/I2C_SCK
- net SCL: now also J2.2; no longer U4.SCL
- net SDA: now also J2.1; no longer U4.SDA
- net TXD.FT: now also R17.1, U3.TXD; no longer R21.1, U5.TXD
- net TXD.NRF: now also R18.2; no longer R22.2
- net TXLED: now also U3.CBUS2; no longer U5.CBUS2
- net USB+: now also C13.1, R12.1; no longer C23.1, R18.1
- net USB-: now also C11.2, R11.1; no longer C24.2, R17.1
- net VIN: now also D1.C; no longer C21.2, C5.2, CHRG2.VIN, D4.C, LDO2.EN, LDO2.IN, R12.2
- net VLIPO: now also D1.A, J1.2, R6.2; no longer C20.1, CHRG2.VBAT, D4.A, J2.2, R13.2
- net V_USB: now also U3.VCC; no longer U5.VCC
Other:
- note added: "Connection to bottom board"
- note removed: "Back-up battery if desired"
- note removed: "I2C Address = 0x68h"
- moved on the sheet: C11, C12, C13, C14, C17, C19, C20, C21, C5, C8, C9, D1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

Commit message: Update 2703-1
Connections:
- removed net A4/BATTERY_STATUS: R6.1, R7.2, U1.P0.28/AIN4
- removed net A6/TIA: J2.6, U1.P0.30/AIN6
- removed net A7/PPG: J2.7, U1.P0.31/AIN7
- removed net D29/LED.CONTROL: J2.5, U1.P0.29/AIN5
- new net A4/PPG: J2.7, U1.P0.28/AIN4
- new net A5/TIA: J2.6, U1.P0.29/AIN5
- new net A7/BATTERY_STATUS: R6.1, R7.2, U1.P0.31/AIN7
- new net D30/LED_CONTROL: J2.5, U1.P0.30/AIN6
Other:
- moved on the sheet: D1, D2, J1, J2, R6, R7, SD1, SW3, SW4, USB1

Commit message: End of class update
Parts:
- removed C10, C9: 300p, LinnesLab-Passives:CAPACITOR0603
- removed SD1: (no value), LinnesLab-Connectors:MICROSD
Connections:
- removed net !DTR: U3.!DTR
- removed net CD2: SD1.CARD_DETECT1
- net 3.3V: no longer SD1.VDD
- net D5/CD1: no longer SD1.CARD_DETECT
- net D7/SD.CS: no longer SD1.CS
- net DTR: now also U3.!DTR
- net GND: no longer C10.2, C9.2, SD1.GND, SD1.GND1, SD1.VSS
- net MISO: no longer SD1.DATA_OUT
- net MOSI: no longer SD1.DATA_IN
- net P0.09/NFC1: no longer C9.1
- net P0.10/NFC2: no longer C10.1
- net SCK: no longer SD1.SCLK
Other:
- note removed: "Connect MISO, MOSI, and SCK to appropriate pins on microcontroller. Those are SPI pins and are generally prespecified. You have more flexibility with the SD.CS pin."
