File: Hardware/Plus/Bottom/Omni-BASIC-BOTTOM.brd (EAGLE design)
At the start: 33 x 33 mm, 36 parts, among them U2 PCF8523

Commit message: 3rd April Update 1
Parts:
- R16: value 1k -> (none)
Changed lines of the file:
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@@
 <attribute name="VALUE" x="30.17096875" y="17.855853125" size="1.27" layer="27" rot="R270"/>
 </element>
-<element name="R16" library="LinnesLab-Passives" package="R0603" package3d_urn="urn:adsk.eagle:package:15661944/2" value="1k" x="19.016978125" y="28.531821875" smashed="yes">
+<element name="R16" library="LinnesLab-Passives" package="R0603" package3d_urn="urn:adsk.eagle:package:15661944/2" value="" x="19.016978125" y="28.531821875" smashed="yes">
 <attribute name="NAME" x="15.8394375" y="28.348940625" size="0.6604" layer="25"/>
 <attribute name="VALUE" x="18.381978125" y="26.626821875" size="1.27" layer="27"/>
