File: Hardware/Plus/Bottom/Omni-BASIC-BOTTOM.sch (EAGLE design)
At the start: 36 parts, among them U2 PCF8523

Commit message: 3rd April Update 1
Parts:
- R16: value 1k -> (none)
Changed lines of the file:
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@@
 <part name="R15" library="LinnesLab-Passives" deviceset="RESISTOR" device="0603" package3d_urn="urn:adsk.eagle:package:15661944/2" value="220k"/>
 <part name="GND17" library="LinnesLab-Symbols" deviceset="GND" device=""/>
-<part name="R16" library="LinnesLab-Passives" deviceset="RESISTOR" device="0603" package3d_urn="urn:adsk.eagle:package:15661944/2" value="1k"/>
+<part name="R16" library="LinnesLab-Passives" deviceset="RESISTOR" device="0603" package3d_urn="urn:adsk.eagle:package:15661944/2"/>
 <part name="GND18" library="CalvEngIO-Symbols" deviceset="GND" device=""/>
 <part name="OP3" library="LinnesLab-AnalogIC" deviceset="OP-QUAD" device="-SO14" package3d_urn="urn:adsk.eagle:package:17879189/2"/>
