File: Hardware/Plus/Top/Omni-BASIC-TOP.sch (EAGLE design)
At the start: 58 parts, among them SW2 SWITCH.MOM, SW3 SWITCH.MOM, U1 NRF52832_MODULE_MDBT42, U3 FT231XS

Commit message: 3rd April Update 1
Changed lines of the file:
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@@
 way dynamically.</text>
 <text x="-154.94" y="396.24" size="1.778" layer="91" grouprefs="CONNECTORS">Connection to bottom board</text>
-<text x="-302.26" y="213.36" size="6.4516" layer="91">Omni Basic Top
+<text x="-312.42" y="152.4" size="6.4516" layer="91">Omni Basic Top
 Revision A
 Date: 03042021
